File: ph_shield_sim7000_pm2_hw/ph_shield_sim7000_pm2_hw.sch (KiCad schematic (older format))
At the start: 83 parts, among them J1 Conn_01x04, J2 Conn_01x07, J3 Conn_01x04, J4 USB_OTG, J5 I2C, J6 Conn_01x10, J7 SIM_Card, Q1 C1815, Q2 C1815, Q3 C1815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

Commit message: door_fume_hood
Parts:
- removed AE3: Antenna, VinhTho_Lib:Anten_GSM_IPEX, symbol ph_shield_sim7000_pm2_hw-rescue:Antenna-Device
- added AE3: Antenna_Shield, VinhTho_Lib:Anten_GSM_IPEX, symbol ph_shield_sim7000_pm2_hw-rescue:Antenna_Shield-Device
Connections:
- net GND: now also AE3.2 (Shield)
- net at C13.1, C14.2, L3.1: now also AE3.1 (A)
Changed lines of the file:
@@
 EESchema Schematic File Version 4
 LIBS:ph_shield_sim7000_pm2_hw-cache
-EELAYER 30 0
+EELAYER 29 0
 EELAYER END
 $Descr A4 11693 8268
@@
 	7325 2300 7325 2250
 Wire Wire Line
-	7800 1825 7800 1925
+	7800 1635 7800 1925
 Wire Wire Line
 	8375 1175 8375 1925
@@
 F 3 "~" H 7075 975 50  0001 C CNN
 	1    7075 875
-	1    0    0    -1
-$EndComp
-$Comp
-L ph_shield_sim7000_pm2_hw-rescue:Antenna-Device AE3
-U 1 1 5E569EF6
-P 7800 1625
-F 0 "AE3" H 7880 1616 50  0000 L CNN
-F 1 "Antenna" H 7880 1525 50  0000 L CNN
-F 2 "VinhTho_Lib:Anten_GSM_IPEX" H 7800 1625 50  0001 C CNN
-F 3 "https://hshop.vn/products/dau-noi-ipex-2" H 7800 1625 50  0001 C CNN
-	1    7800 1625
 	1    0    0    -1
 $EndComp
@@
 	1    0    0    -1
 $EndComp
+$Comp
+L ph_shield_sim7000_pm2_hw-rescue:Antenna_Shield-Device AE3
+U 1 1 5DBD87BF
+P 7800 1435
+F 0 "AE3" H 7940 1476 50  0000 L CNN
+F 1 "Antenna_Shield" H 7940 1385 50  0000 L CNN
+F 2 "VinhTho_Lib:Anten_GSM_IPEX" H 7800 1535 50  0001 C CNN
+F 3 "https://hshop.vn/products/dau-noi-ipex-2" H 7800 1535 50  0001 C CNN
+	1    7800 1435
+	1    0    0    -1
+$EndComp
+$Comp
+L ph_shield_sim7000_pm2_hw-rescue:GND-power #PWR?
+U 1 1 5DBDA6CD
+P 7900 1665
+F 0 "#PWR?" H 7900 1415 50  0001 C CNN
+F 1 "GND" H 7905 1492 50  0000 C CNN
+F 2 "" H 7900 1665 50  0001 C CNN
+F 3 "" H 7900 1665 50  0001 C CNN
+	1    7900 1665
+	1    0    0    -1
+$EndComp
+Wire Wire Line
+	7900 1635 7900 1665
 $EndSCHEMATC
