File: ph_door_fume_hood_controller_hw/ph_door_fume_hood_controller_hw.sch (KiCad schematic (older format))
At the start: 250 parts, among them IC1 6N137, J1 Conn_01x03, J10 Conn_01x04, J11 Conn_01x02, J2 Conn_01x03, J3 USB_OTG, J4 CONN_01X04, J5 Conn_01x03, J6 Conn_01x06, J7 Conn_01x03, J8 Conn_01x03, J9 Conn_01x02, M1 MORSUN_485, M2 DC-DC-24-12V-200mA, Q1 C1815, Q2 Q_NMOS_GDS, U1 ASM1117-3V3, U10 AD8601, U11 PC817, U12 PC817, U13 74HC123, U14 ASM1117, U15 XL4015, U16 TB6600, U2 PC817, U3 PC817, U4 STM32F103C8, U5 PC817, U6 PC817, U7 PC817, U8 PC817, U9 PC817, Y1 Crystal, Y2 32768Mhz

Commit message: Darwing board fume hood
Parts:
- BT1: footprint Pin_Headers:Pin_Header_Straight_1x02_Pitch2.54mm -> VinhTho_Lib:BT3V3
- C1: renamed from C28; footprint Capacitors_SMD:C_0805_HandSoldering -> Capacitor_SMD:C_0805_2012Metric_Pad1.15x1.40mm_HandSolder
- C10: renamed from C16; footprint Capacitors_SMD:C_0805_HandSoldering -> Capacitor_SMD:C_0805_2012Metric_Pad1.15x1.40mm_HandSolder
- C11: renamed from C21; footprint Capacitors_SMD:C_0805_HandSoldering -> Capacitor_SMD:C_0805_2012Metric_Pad1.15x1.40mm_HandSolder
- C12: renamed from C22; footprint Capacitors_SMD:C_0805_HandSoldering -> Capacitor_SMD:C_0805_2012Metric_Pad1.15x1.40mm_HandSolder
- C13: renamed from C23; footprint Capacitors_SMD:C_1206_HandSoldering -> Capacitor_SMD:C_1206_3216Metric_Pad1.42x1.75mm_HandSolder
- C14: renamed from C10; footprint Capacitors_SMD:C_0805_HandSoldering -> Capacitor_SMD:C_0805_2012Metric_Pad1.15x1.40mm_HandSolder
- C15: renamed from C34; footprint Capacitors_SMD:C_0805_HandSoldering -> Capacitor_SMD:C_0805_2012Metric_Pad1.15x1.40mm_HandSolder
- C16, C35, C37, C45, C46: renamed from C?; footprint Capacitors_SMD:C_0805_HandSoldering -> Capacitor_SMD:C_0805_2012Metric_Pad1.15x1.40mm_HandSolder
- C17: renamed from C11; footprint Capacitors_SMD:C_0805_HandSoldering -> Capacitor_SMD:C_0805_2012Metric_Pad1.15x1.40mm_HandSolder
- C18: renamed from C24; footprint Capacitors_SMD:C_0805_HandSoldering -> Capacitor_SMD:C_0805_2012Metric_Pad1.15x1.40mm_HandSolder
- C19: renamed from C12; footprint Capacitors_SMD:C_0805_HandSoldering -> Capacitor_SMD:C_0805_2012Metric_Pad1.15x1.40mm_HandSolder
- C2: renamed from C29; footprint Capacitors_SMD:C_1206_HandSoldering -> Capacitor_SMD:C_1206_3216Metric_Pad1.42x1.75mm_HandSolder
- C20: renamed from C35; footprint Capacitors_SMD:C_0805_HandSoldering -> Capacitor_SMD:C_0805_2012Metric_Pad1.15x1.40mm_HandSolder
- C21: renamed from C17; footprint Capacitors_SMD:C_0805_HandSoldering -> Capacitor_SMD:C_0805_2012Metric_Pad1.15x1.40mm_HandSolder
- C22: renamed from C13; footprint Capacitors_SMD:C_0805_HandSoldering -> Capacitor_SMD:C_0805_2012Metric_Pad1.15x1.40mm_HandSolder
- C23: renamed from C18; footprint Capacitors_SMD:C_0805_HandSoldering -> Capacitor_SMD:C_0805_2012Metric_Pad1.15x1.40mm_HandSolder
- C24: renamed from C26; footprint Capacitors_SMD:C_0805_HandSoldering -> Capacitor_SMD:C_0805_2012Metric_Pad1.15x1.40mm_HandSolder
- C25: renamed from C27; footprint Capacitors_SMD:C_0805_HandSoldering -> Capacitor_SMD:C_0805_2012Metric_Pad1.15x1.40mm_HandSolder
- C26: renamed from C32; footprint Capacitors_SMD:C_0805_HandSoldering -> Capacitor_SMD:C_0805_2012Metric_Pad1.15x1.40mm_HandSolder
- C27: renamed from C33; footprint Capacitors_SMD:C_1210_HandSoldering -> Capacitor_SMD:C_1210_3225Metric_Pad1.42x2.65mm_HandSolder
- C28: renamed from C40; footprint Capacitors_SMD:C_0805_HandSoldering -> Capacitor_SMD:C_0805_2012Metric_Pad1.15x1.40mm_HandSolder
- C29: renamed from C30; footprint Capacitors_SMD:C_0805_HandSoldering -> Capacitor_SMD:C_0805_2012Metric_Pad1.15x1.40mm_HandSolder
- C3: renamed from C37; footprint Capacitors_SMD:C_1206_HandSoldering -> Capacitor_SMD:C_1206_3216Metric_Pad1.42x1.75mm_HandSolder
- C30: renamed from C31; footprint Capacitors_SMD:C_0805_HandSoldering -> Capacitor_SMD:C_0805_2012Metric_Pad1.15x1.40mm_HandSolder
- C31: renamed from C42; footprint Capacitors_SMD:C_0805_HandSoldering -> Capacitor_SMD:C_0805_2012Metric_Pad1.15x1.40mm_HandSolder
- C32: renamed from C44; footprint Capacitors_SMD:C_1210_HandSoldering -> Capacitor_SMD:C_1210_3225Metric_Pad1.42x2.65mm_HandSolder
- C33: renamed from C20; footprint Capacitors_SMD:C_0805_HandSoldering -> Capacitor_SMD:C_0805_2012Metric_Pad1.15x1.40mm_HandSolder
- C34: renamed from C25; footprint Capacitors_SMD:C_1210_HandSoldering -> Capacitor_SMD:C_1210_3225Metric_Pad1.42x2.65mm_HandSolder
- C36: renamed from C15; footprint Capacitors_SMD:C_0805_HandSoldering -> Capacitor_SMD:C_0805_2012Metric_Pad1.15x1.40mm_HandSolder
- C38: renamed from C36; footprint Capacitors_SMD:C_0805_HandSoldering -> Capacitor_SMD:C_0805_2012Metric_Pad1.15x1.40mm_HandSolder
- C39: footprint Capacitors_SMD:C_1210_HandSoldering -> Capacitor_SMD:C_1210_3225Metric_Pad1.42x2.65mm_HandSolder
- C4: renamed from C38; footprint Capacitors_SMD:C_0805_HandSoldering -> Capacitor_SMD:C_0805_2012Metric_Pad1.15x1.40mm_HandSolder
- C40: renamed from C4; footprint Capacitors_SMD:C_0805_HandSoldering -> Capacitor_SMD:C_0805_2012Metric_Pad1.15x1.40mm_HandSolder
- C41: renamed from C5; footprint Capacitors_SMD:C_1210_HandSoldering -> Capacitor_SMD:C_1210_3225Metric_Pad1.42x2.65mm_HandSolder
- C42: renamed from C6; footprint Capacitors_SMD:C_0805_HandSoldering -> Capacitor_SMD:C_0805_2012Metric_Pad1.15x1.40mm_HandSolder
- C43: renamed from C46; footprint Capacitors_SMD:C_0805_HandSoldering -> Capacitor_SMD:C_0805_2012Metric_Pad1.15x1.40mm_HandSolder
- C44: renamed from C47; footprint Capacitors_SMD:C_1210_HandSoldering -> Capacitor_SMD:C_1210_3225Metric_Pad1.42x2.65mm_HandSolder
- C47: renamed from C7; footprint Capacitors_SMD:C_0805_HandSoldering -> Capacitor_SMD:C_0805_2012Metric_Pad1.15x1.40mm_HandSolder
- C48: renamed from C3; footprint Capacitors_SMD:C_0805_HandSoldering -> Capacitor_SMD:C_0805_2012Metric_Pad1.15x1.40mm_HandSolder
- C49: renamed from C8; footprint Capacitors_SMD:C_0805_HandSoldering -> Capacitor_SMD:C_0805_2012Metric_Pad1.15x1.40mm_HandSolder
- C5: renamed from C45; footprint Capacitors_SMD:C_1210_HandSoldering -> Capacitor_SMD:C_1210_3225Metric_Pad1.42x2.65mm_HandSolder
- C50: renamed from C1; footprint Capacitors_SMD:C_0805_HandSoldering -> Capacitor_SMD:C_0805_2012Metric_Pad1.15x1.40mm_HandSolder
- C51: renamed from C9; footprint Capacitors_SMD:C_0805_HandSoldering -> Capacitor_SMD:C_0805_2012Metric_Pad1.15x1.40mm_HandSolder
- C52: renamed from C2; footprint Capacitors_SMD:C_0805_HandSoldering -> Capacitor_SMD:C_0805_2012Metric_Pad1.15x1.40mm_HandSolder
- C6: renamed from C14; footprint Capacitors_SMD:C_0805_HandSoldering -> Capacitor_SMD:C_0805_2012Metric_Pad1.15x1.40mm_HandSolder
- C7: renamed from C41; footprint Capacitors_SMD:C_0805_HandSoldering -> Capacitor_SMD:C_0805_2012Metric_Pad1.15x1.40mm_HandSolder
- C8: renamed from C43; footprint Capacitors_SMD:C_0805_HandSoldering -> Capacitor_SMD:C_0805_2012Metric_Pad1.15x1.40mm_HandSolder
- C9: renamed from C19; footprint Capacitors_SMD:C_0805_HandSoldering -> Capacitor_SMD:C_0805_2012Metric_Pad1.15x1.40mm_HandSolder
- D1: renamed from D16; footprint LEDs:LED_0805 -> LED_SMD:LED_0805_2012Metric_Pad1.15x1.40mm_HandSolder
- D10, D16, D22, D26, D30: renamed from D?; footprint (none) -> VinhTho_Lib:D_SMA_Standard
- D11: renamed from D19; footprint nhantt-kicad-lib:D_SMA_Standard -> VinhTho_Lib:D_SMA_Standard
- D12, D18, D24, D29, D33: renamed from D?; footprint (none) -> VinhTho_Lib:SOD-80
- D13: renamed from D4; footprint Diodes_SMD:D_SOD-123F -> VinhTho_Lib:D_SOD-323F
- D14, D5, D6: renamed from D?; footprint LEDs:LED_0805 -> LED_SMD:LED_0805_2012Metric_Pad1.15x1.40mm_HandSolder
- D15: renamed from D7; footprint nhantt-kicad-lib:D_SOD-323F -> VinhTho_Lib:D_SOD-323F
- D17: renamed from D8; footprint (none) -> VinhTho_Lib:D_SMA_Standard
- D19: renamed from D11; footprint (none) -> VinhTho_Lib:D_SMA_Standard
- D2: renamed from D17; footprint LEDs:LED_0805 -> LED_SMD:LED_0805_2012Metric_Pad1.15x1.40mm_HandSolder
- D20: renamed from D1; footprint (none) -> VinhTho_Lib:D_SMA_Standard
- D21: renamed from D9; footprint nhantt-kicad-lib:D_SMA_Standard -> VinhTho_Lib:D_SMA_Standard
- D23: renamed from D15; footprint nhantt-kicad-lib:D_SMA_Standard -> VinhTho_Lib:D_SMA_Standard
- D25: renamed from D10; footprint nhantt-kicad-lib:D_SMA_Standard -> VinhTho_Lib:D_SMA_Standard
- D27: renamed from D12; footprint (none) -> VinhTho_Lib:D_SMA_Standard
- D28: renamed from D3; footprint (none) -> VinhTho_Lib:D_SMA_Standard
- D3: renamed from D14; footprint Diode_THT:D_DO-35_SOD27_P7.62mm_Horizontal -> Diode_SMD:D_SOD-323_HandSoldering
- D31: renamed from D13; footprint (none) -> VinhTho_Lib:D_SMA_Standard
- D32: renamed from D5; footprint (none) -> VinhTho_Lib:D_SMA_Standard
- D4: renamed from D6; footprint LEDs:LED_0805 -> LED_SMD:LED_0805_2012Metric_Pad1.15x1.40mm_HandSolder
- D7: renamed from D20; footprint nhantt-kicad-lib:D_SMA_Standard -> VinhTho_Lib:D_SMA_Standard
- D8: renamed from D2; footprint LEDs:LED_0805 -> LED_SMD:LED_0805_2012Metric_Pad1.15x1.40mm_HandSolder
- D9: renamed from D18; footprint nhantt-kicad-lib:D_SMA_Standard -> VinhTho_Lib:D_SMA_Standard
- F1: footprint (none) -> VinhTho_Lib:Fuse_SMD1812
- F2, F3, F4, F7: renamed from F?; footprint (none) -> VinhTho_Lib:Fuse_SMD1812
- F5: renamed from F2; footprint nhantt-kicad-lib:Fuse_SMD1812 -> VinhTho_Lib:Fuse_SMD1812
- F6: renamed from F3; footprint nhantt-kicad-lib:Fuse_SMD1812 -> VinhTho_Lib:Fuse_SMD1812
- IC1: footprint nhantt-kicad-lib:Diodes_PSOP-8 -> VinhTho_Lib:Diodes_PSOP-8
- IC2: renamed from IC?; footprint nhantt-kicad-lib:Diodes_PSOP-8 -> VinhTho_Lib:Diodes_PSOP-8
- J2: renamed from J10; footprint (none) -> VinhTho_Lib:Domino-5.08mm_4pol
- J8: renamed from J3; footprint nhantt-kicad-lib:USB_Micro-B -> VinhTho_Lib:USB_Micro-B
- L1: renamed from L2; footprint Inductors_SMD:L_0805_HandSoldering -> Inductor_SMD:L_0805_2012Metric_Pad1.15x1.40mm_HandSolder
- L2: renamed from L1; value L_Core_Ferrite -> 180uH/5A; footprint (none) -> VinhTho_Lib:L181-5A
- LS1: footprint nhantt-kicad-lib:SMD_BUZZER_9633 -> VinhTho_Lib:SMD_BUZZER_9633
- M2: renamed from M1; footprint (none) -> VinhTho_Lib:MORSUN_485
- Q1, Q10, Q8: renamed from Q?; footprint nhantt-kicad-lib:SOT-23 -> VinhTho_Lib:SOT-23
- Q5: renamed from Q1; footprint nhantt-kicad-lib:SOT-23 -> VinhTho_Lib:SOT-23
- R1, R12, R13, R2, R25, R33, R4, R46, R48, R5, R50, R51, R52, R53, R56, R58, R61, R63, R65, R67, R68, R69, R71, R75, R76, R77, R79, R8, R80, R82, R86, R87, R88, R89, R9, R90, R93, R96: renamed from R?; footprint Resistors_SMD:R_0805_HandSoldering -> Resistor_SMD:R_0805_2012Metric_Pad1.15x1.40mm_HandSolder
- R10: renamed from R32; footprint Resistors_SMD:R_0805_HandSoldering -> Resistor_SMD:R_0805_2012Metric_Pad1.15x1.40mm_HandSolder
- R11: renamed from R49; footprint Resistors_SMD:R_0805_HandSoldering -> Resistor_SMD:R_0805_2012Metric_Pad1.15x1.40mm_HandSolder
- R14: renamed from R27; footprint Resistors_SMD:R_0805_HandSoldering -> Resistor_SMD:R_0805_2012Metric_Pad1.15x1.40mm_HandSolder
- R15: renamed from R38; footprint Resistors_SMD:R_0805_HandSoldering -> Resistor_SMD:R_0805_2012Metric_Pad1.15x1.40mm_HandSolder
- R16: renamed from R40; footprint Resistors_SMD:R_0805_HandSoldering -> Resistor_SMD:R_0805_2012Metric_Pad1.15x1.40mm_HandSolder
- R17: renamed from R44; footprint Resistors_SMD:R_0805_HandSoldering -> Resistor_SMD:R_0805_2012Metric_Pad1.15x1.40mm_HandSolder
- R18: renamed from R24; footprint Resistors_SMD:R_0805_HandSoldering -> Resistor_SMD:R_0805_2012Metric_Pad1.15x1.40mm_HandSolder
- R19: renamed from R31; footprint Resistors_SMD:R_0805_HandSoldering -> Resistor_SMD:R_0805_2012Metric_Pad1.15x1.40mm_HandSolder
- R20: renamed from R23; footprint Resistors_SMD:R_0805_HandSoldering -> Resistor_SMD:R_0805_2012Metric_Pad1.15x1.40mm_HandSolder
- R21: renamed from R39; footprint Resistors_SMD:R_0805_HandSoldering -> Resistor_SMD:R_0805_2012Metric_Pad1.15x1.40mm_HandSolder
- R22: renamed from R41; footprint Resistors_SMD:R_0805_HandSoldering -> Resistor_SMD:R_0805_2012Metric_Pad1.15x1.40mm_HandSolder
- R23: renamed from R45; footprint Resistors_SMD:R_0805_HandSoldering -> Resistor_SMD:R_0805_2012Metric_Pad1.15x1.40mm_HandSolder
- R24: renamed from R33; footprint Resistors_SMD:R_0805_HandSoldering -> Resistor_SMD:R_0805_2012Metric_Pad1.15x1.40mm_HandSolder
- R26: renamed from R25; footprint Resistors_SMD:R_0805_HandSoldering -> Resistor_SMD:R_0805_2012Metric_Pad1.15x1.40mm_HandSolder
- R27: renamed from R28; footprint Resistors_SMD:R_0805_HandSoldering -> Resistor_SMD:R_0805_2012Metric_Pad1.15x1.40mm_HandSolder
- R28: renamed from R52; footprint Resistors_SMD:R_0805_HandSoldering -> Resistor_SMD:R_0805_2012Metric_Pad1.15x1.40mm_HandSolder
- R29: renamed from R54; footprint Resistors_SMD:R_0805_HandSoldering -> Resistor_SMD:R_0805_2012Metric_Pad1.15x1.40mm_HandSolder
- R3: renamed from R50; footprint Resistors_SMD:R_0805_HandSoldering -> Resistor_SMD:R_0805_2012Metric_Pad1.15x1.40mm_HandSolder
- R30: renamed from R56; footprint Resistors_SMD:R_0805_HandSoldering -> Resistor_SMD:R_0805_2012Metric_Pad1.15x1.40mm_HandSolder
- R31: renamed from R42; footprint Resistors_SMD:R_0805_HandSoldering -> Resistor_SMD:R_0805_2012Metric_Pad1.15x1.40mm_HandSolder
- R32: renamed from R34; footprint Resistors_SMD:R_0805_HandSoldering -> Resistor_SMD:R_0805_2012Metric_Pad1.15x1.40mm_HandSolder
- R34: renamed from R36; footprint Resistors_SMD:R_0805_HandSoldering -> Resistor_SMD:R_0805_2012Metric_Pad1.15x1.40mm_HandSolder
- R35: renamed from R5; footprint Resistors_SMD:R_0805_HandSoldering -> Resistor_SMD:R_0805_2012Metric_Pad1.15x1.40mm_HandSolder
- R36: renamed from R35; footprint Resistors_SMD:R_0805_HandSoldering -> Resistor_SMD:R_0805_2012Metric_Pad1.15x1.40mm_HandSolder
- R37: renamed from R29; footprint Resistors_SMD:R_0805_HandSoldering -> Resistor_SMD:R_0805_2012Metric_Pad1.15x1.40mm_HandSolder
- R38: renamed from R43; footprint Resistors_SMD:R_0805_HandSoldering -> Resistor_SMD:R_0805_2012Metric_Pad1.15x1.40mm_HandSolder
- R39: renamed from R51; footprint Resistors_SMD:R_0805_HandSoldering -> Resistor_SMD:R_0805_2012Metric_Pad1.15x1.40mm_HandSolder
- R40: renamed from R53; footprint Resistors_SMD:R_0805_HandSoldering -> Resistor_SMD:R_0805_2012Metric_Pad1.15x1.40mm_HandSolder
- R41: renamed from R55; footprint Resistors_SMD:R_0805_HandSoldering -> Resistor_SMD:R_0805_2012Metric_Pad1.15x1.40mm_HandSolder
- R42: renamed from R37; footprint Resistors_SMD:R_0805_HandSoldering -> Resistor_SMD:R_0805_2012Metric_Pad1.15x1.40mm_HandSolder
- R43: renamed from R48; footprint Resistors_SMD:R_0805_HandSoldering -> Resistor_SMD:R_0805_2012Metric_Pad1.15x1.40mm_HandSolder
- R44: renamed from R6; footprint Resistors_SMD:R_0805_HandSoldering -> Resistor_SMD:R_0805_2012Metric_Pad1.15x1.40mm_HandSolder
- R45: renamed from R2; footprint Resistors_SMD:R_0805_HandSoldering -> Resistor_SMD:R_0805_2012Metric_Pad1.15x1.40mm_HandSolder
- R47: renamed from R46; footprint Resistors_SMD:R_0805_HandSoldering -> Resistor_SMD:R_0805_2012Metric_Pad1.15x1.40mm_HandSolder
- R49: renamed from R47; footprint Resistors_SMD:R_0805_HandSoldering -> Resistor_SMD:R_0805_2012Metric_Pad1.15x1.40mm_HandSolder
- R54: renamed from R10; footprint Resistors_SMD:R_0805_HandSoldering -> Resistor_SMD:R_0805_2012Metric_Pad1.15x1.40mm_HandSolder
- R55: renamed from R14; footprint Resistors_SMD:R_0805_HandSoldering -> Resistor_SMD:R_0805_2012Metric_Pad1.15x1.40mm_HandSolder
- R57: renamed from R17; footprint Resistors_SMD:R_0805_HandSoldering -> Resistor_SMD:R_0805_2012Metric_Pad1.15x1.40mm_HandSolder
- R59, R60: renamed from R?; footprint Resistors_SMD:R_2512_HandSoldering -> Resistor_SMD:R_0805_2012Metric_Pad1.15x1.40mm_HandSolder
- R6: renamed from R26; footprint Resistors_SMD:R_0805_HandSoldering -> Resistor_SMD:R_0805_2012Metric_Pad1.15x1.40mm_HandSolder
- R62: renamed from R16; footprint Resistors_SMD:R_0805_HandSoldering -> Resistor_SMD:R_0805_2012Metric_Pad1.15x1.40mm_HandSolder
- R64: renamed from R22; footprint Resistors_SMD:R_0805_HandSoldering -> Resistor_SMD:R_0805_2012Metric_Pad1.15x1.40mm_HandSolder
- R66: renamed from R11; footprint Resistors_SMD:R_0805_HandSoldering -> Resistor_SMD:R_0805_2012Metric_Pad1.15x1.40mm_HandSolder
- R7: renamed from R30; footprint Resistors_SMD:R_0805_HandSoldering -> Resistor_SMD:R_0805_2012Metric_Pad1.15x1.40mm_HandSolder
- R70: renamed from R18; footprint Resistors_SMD:R_0805_HandSoldering -> Resistor_SMD:R_0805_2012Metric_Pad1.15x1.40mm_HandSolder
- R72: renamed from R7; footprint Resistors_SMD:R_0805_HandSoldering -> Resistor_SMD:R_0805_2012Metric_Pad1.15x1.40mm_HandSolder
- R73: renamed from R12; footprint Resistors_SMD:R_0805_HandSoldering -> Resistor_SMD:R_0805_2012Metric_Pad1.15x1.40mm_HandSolder
- R74: renamed from R1; footprint Resistors_SMD:R_0805_HandSoldering -> Resistor_SMD:R_0805_2012Metric_Pad1.15x1.40mm_HandSolder
- R78: renamed from R20; footprint Resistors_SMD:R_0805_HandSoldering -> Resistor_SMD:R_0805_2012Metric_Pad1.15x1.40mm_HandSolder
- R81: renamed from R19; footprint Resistors_SMD:R_0805_HandSoldering -> Resistor_SMD:R_0805_2012Metric_Pad1.15x1.40mm_HandSolder
- R83: renamed from R8; footprint Resistors_SMD:R_0805_HandSoldering -> Resistor_SMD:R_0805_2012Metric_Pad1.15x1.40mm_HandSolder
- R84: renamed from R13; footprint Resistors_SMD:R_0805_HandSoldering -> Resistor_SMD:R_0805_2012Metric_Pad1.15x1.40mm_HandSolder
- R85: renamed from R3; footprint Resistors_SMD:R_0805_HandSoldering -> Resistor_SMD:R_0805_2012Metric_Pad1.15x1.40mm_HandSolder
- R91: renamed from R21; footprint Resistors_SMD:R_0805_HandSoldering -> Resistor_SMD:R_0805_2012Metric_Pad1.15x1.40mm_HandSolder
- R92: renamed from R9; footprint Resistors_SMD:R_0805_HandSoldering -> Resistor_SMD:R_0805_2012Metric_Pad1.15x1.40mm_HandSolder
- R94: renamed from R15; footprint Resistors_SMD:R_0805_HandSoldering -> Resistor_SMD:R_0805_2012Metric_Pad1.15x1.40mm_HandSolder
- R95: renamed from R4; footprint Resistors_SMD:R_0805_HandSoldering -> Resistor_SMD:R_0805_2012Metric_Pad1.15x1.40mm_HandSolder
- RV1: footprint (none) -> VinhTho_Lib:VR1
- U1: renamed from U13; footprint (none) -> VinhTho_Lib:SOIC-16W_5.3x10.2mm_Pitch1.27mm
- U11: renamed from U?; footprint nhantt-kicad-lib:SOT-23-6_Handsoldering -> VinhTho_Lib:SOT-23-6_Handsoldering
- U12: renamed from U1; footprint nhantt-kicad-lib:SOT-223 -> VinhTho_Lib:SOT-223
- U15: renamed from U?; footprint (none) -> Package_SO:SOP-8_3.76x4.96mm_P1.27mm
- U2: renamed from U10; footprint nhantt-kicad-lib:SOT-23-5 -> VinhTho_Lib:SOT-23-5
- U5: renamed from U16; footprint (none) -> VinhTho_Lib:TB6600
- U7: renamed from U4; footprint nhantt-kicad-lib:LQFP-48_7x7mm_Pitch0.5mm -> VinhTho_Lib:LQFP-48_7x7mm_Pitch0.5mm
- U8: renamed from U14; footprint st-kicad-lib:SOT-223 -> VinhTho_Lib:SOT-223
- U9: renamed from U15; footprint TO_SOT_Packages_SMD:TO-263-5_TabPin3 -> Package_TO_SOT_SMD:TO-263-5_TabPin3
- Y1: footprint Crystals:Crystal_SMD_5032-2pin_5.0x3.2mm_HandSoldering -> VinhTho_Lib:Crystal_SMD_HC49-SD
- Y2: footprint Crystals:Crystal_SMD_3215-2pin_3.2x1.5mm -> VinhTho_Lib:Crystal_Round_Horizontal_3mm_smd
- gave numbers to parts that had none: 16
- renumbered J7 to J1, J1 to J10, J9 to J11, J6 to J12, J2 to J14, J5 to J15, J4 to J3, J8 to J4, J11 to J6, M2 to M1, Q2 to Q3, U6 to U14, U7 to U16, U2 to U17, U8 to U19, U3 to U20, U9 to U22, U5 to U23, U11 to U4, U12 to U6

Commit message: Layoutting board fume_hood
Parts:
- D17, D19, D20, D27, D28, D31, D32: footprint VinhTho_Lib:D_SMA_Standard -> VinhTho_Lib:SOD-80
- J1, J10, J14, J15, J4, J5: footprint (none) -> VinhTho_Lib:TerminalBlock-WAGO-3P
- J11, J13, J6, J9: footprint (none) -> VinhTho_Lib:TerminalBlock_WAGO-236_2Stift_R5mm_2pol
- J12, J7: footprint (none) -> VinhTho_Lib:TerminalBlock-WAGO-6P
- J3: footprint Pin_Headers:Pin_Header_Straight_1x04_Pitch2.54mm -> Connector_PinHeader_2.54mm:PinHeader_1x04_P2.54mm_Vertical
- LS1: footprint VinhTho_Lib:SMD_BUZZER_9633 -> Buzzer_Beeper:Buzzer_15x7.5RM7.6
- M1: footprint nhantt-kicad-lib:muRata2405 -> VinhTho_Lib:MORNSUN-A2412S-2W
- Q11, Q2, Q3, Q4, Q6, Q7, Q9: footprint (none) -> VinhTho_Lib:TO-252-2
- R59, R60: footprint Resistor_SMD:R_0805_2012Metric_Pad1.15x1.40mm_HandSolder -> Resistor_SMD:R_2512_6332Metric_Pad1.52x3.35mm_HandSolder
Connections:
- net GND: now also M1.5 (0V); no longer M1.4 (Vo-)
- net +24V: now reaches R46.1
- net +24V: now also C28.1, C31.1, C32.1, C43.1, C44.1, D10.1 (K), D16.1 (K), D22.1 (K), D26.1 (K), D30.1 (K), D9.1 (K), J10.1 (Pin_1), J12.1 (Pin_1), J12.2 (Pin_2), J13.1 (Pin_1), J14.1 (Pin_1), J15.1 (Pin_1), J7.1 (Pin_1), J7.2 (Pin_2), M1.1 (Vin+), R61.1, R75.1, R79.1, R89.1, U9.5 (VIN)
