File: ph_door_fume_hood_controller_hw/ph_door_fume_hood_controller_hw.sch (KiCad schematic (older format))
At the start: 247 parts, among them IC1 6N137, IC2 6N137, J1 Conn_01x03, J10 Conn_01x03, J11 Conn_01x02, J12 Conn_01x06, J13 Conn_01x02, J14 Conn_01x03, J15 Conn_01x03, J2 Conn_01x04, J3 CONN_01X04, J4 Conn_01x03, J5 Conn_01x04, J6 Conn_01x02, J7 Conn_01x06, J8 USB_OTG, J9 Conn_01x02, M1 DC-DC-24-12V-200mA, M2 MORSUN_485, Q1 C1815, Q10 A1015, Q11 Q_NMOS_GSD, Q2 Q_PMOS_GDS, Q3 Q_NMOS_GSD, Q4 Q_NMOS_GSD, Q5 C1815, Q6 Q_NMOS_GSD, Q7 Q_NMOS_GSD, Q8 C1815, Q9 Q_NMOS_GSD, U1 74HC123, U10 PC817, U11 MCP4725, U12 ASM1117-3V3, U13 PC817, U14 PC817, U15 LM358, U16 PC817, U17 PC817, U18 PC817, U19 PC817, U2 AD8601, U20 PC817, U21 PC817, U22 PC817, U23 PC817, U3 PC817, U4 PC817, U5 TB6600, U6 PC817, U7 STM32F103C8, U8 ASM1117, U9 XL4015, Y1 Crystal, Y2 32768Mhz

Commit message: Edit power for fume hood
Parts:
- IC1, IC2: Link Mua Hang (none) -> https://banlinhkien.com/6n137-sop8-opto-10mbits-p6650639.ht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
- R28, R29, R30, R39, R40, R41: footprint Resistor_SMD:R_0805_2012Metric_Pad1.15x1.40mm_HandSolder -> Resistor_SMD:R_2512_6332Metric_Pad1.52x3.35mm_HandSolder
Changed lines of the file:
@@
 EESchema Schematic File Version 4
 LIBS:ph_door_fume_hood_controller_hw-cache
-EELAYER 30 0
+EELAYER 29 0
 EELAYER END
 $Descr A3 16535 11693
@@
 F 0 "R28" V 14455 2300 50  0000 C CNN
 F 1 "0.62R" V 14375 2300 50  0000 C CNN
-F 2 "Resistor_SMD:R_0805_2012Metric_Pad1.15x1.40mm_HandSolder" V 14305 2300 50  0001 C CNN
+F 2 "Resistor_SMD:R_2512_6332Metric_Pad1.52x3.35mm_HandSolder" V 14305 2300 50  0001 C CNN
 F 3 "" H 14375 2300 50  0001 C CNN
 	1    14375 2300
@@
 F 0 "R29" V 14605 2300 50  0000 C CNN
 F 1 "0.62R" V 14525 2300 50  0000 C CNN
-F 2 "Resistor_SMD:R_0805_2012Metric_Pad1.15x1.40mm_HandSolder" V 14455 2300 50  0001 C CNN
+F 2 "Resistor_SMD:R_2512_6332Metric_Pad1.52x3.35mm_HandSolder" V 14455 2300 50  0001 C CNN
 F 3 "" H 14525 2300 50  0001 C CNN
 	1    14525 2300
@@
 F 0 "R30" V 14730 2300 50  0000 C CNN
 F 1 "0.62R" V 14650 2300 50  0000 C CNN
-F 2 "Resistor_SMD:R_0805_2012Metric_Pad1.15x1.40mm_HandSolder" V 14580 2300 50  0001 C CNN
+F 2 "Resistor_SMD:R_2512_6332Metric_Pad1.52x3.35mm_HandSolder" V 14580 2300 50  0001 C CNN
 F 3 "" H 14650 2300 50  0001 C CNN
 	1    14650 2300
@@
 F 0 "R39" V 14405 3000 50  0000 C CNN
 F 1 "0.62R" V 14325 3000 50  0000 C CNN
-F 2 "Resistor_SMD:R_0805_2012Metric_Pad1.15x1.40mm_HandSolder" V 14255 3000 50  0001 C CNN
+F 2 "Resistor_SMD:R_2512_6332Metric_Pad1.52x3.35mm_HandSolder" V 14255 3000 50  0001 C CNN
 F 3 "" H 14325 3000 50  0001 C CNN
 	1    14325 3000
@@
 F 0 "R40" V 14530 3000 50  0000 C CNN
 F 1 "0.62R" V 14450 3000 50  0000 C CNN
-F 2 "Resistor_SMD:R_0805_2012Metric_Pad1.15x1.40mm_HandSolder" V 14380 3000 50  0001 C CNN
+F 2 "Resistor_SMD:R_2512_6332Metric_Pad1.52x3.35mm_HandSolder" V 14380 3000 50  0001 C CNN
 F 3 "" H 14450 3000 50  0001 C CNN
 	1    14450 3000
@@
 F 0 "R41" V 14655 3000 50  0000 C CNN
 F 1 "0.62R" V 14575 3000 50  0000 C CNN
-F 2 "Resistor_SMD:R_0805_2012Metric_Pad1.15x1.40mm_HandSolder" V 14505 3000 50  0001 C CNN
+F 2 "Resistor_SMD:R_2512_6332Metric_Pad1.52x3.35mm_HandSolder" V 14505 3000 50  0001 C CNN
 F 3 "" H 14575 3000 50  0001 C CNN
 	1    14575 3000
@@
 F 2 "VinhTho_Lib:Diodes_PSOP-8" H 8735 890 29  0001 C CNN
 F 3 "https://banlinhkien.com/6n137-sop8-opto-10mbits-p6650639.html" H 8686 1354 60  0001 C CNN
+F 4 "https://banlinhkien.com/6n137-sop8-opto-10mbits-p6650639.html" H 8900 1125 50  0001 C CNN "Link Mua Hang"
 	1    8900 1125
 	1    0    0    -1
@@
 F 2 "VinhTho_Lib:Diodes_PSOP-8" H 9810 9165 29  0001 C CNN
 F 3 "https://banlinhkien.com/6n137-sop8-opto-10mbits-p6650639.html" H 9761 9629 60  0001 C CNN
+F 4 "https://banlinhkien.com/6n137-sop8-opto-10mbits-p6650639.html" H 9975 9400 50  0001 C CNN "Link Mua Hang"
 	1    9975 9400
 	1    0    0    -1
@@
 	2750 6375 2750 6425
 $Comp
-L ph_door_fume_hood_controller_hw-rescue:+5VA-power #PWR?
+L ph_door_fume_hood_controller_hw-rescue:+5VA-power #PWR0116
 U 1 1 5DEAC768
 P 525 6050
-F 0 "#PWR?" H 525 5900 50  0001 C CNN
+F 0 "#PWR0116" H 525 5900 50  0001 C CNN
 F 1 "+5VA" H 540 6223 50  0000 C CNN
 F 2 "" H 525 6050 50  0001 C CNN

Commit message: Update
Parts:
- IC2: footprint VinhTho_Lib:Diodes_PSOP-8 -> ph_kicad_lib:SMDIP-8_W9.53mm
- M1: Link Mua Hang (none) -> https://banlinhkien.shop/module-nguon-cach-ly-a2412s-2w-mor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
- Q2: Link Mua Hang (none) -> https://banlinhkien.com/d409-to252-mosfet-pch-26a-60v-p6650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
- RV1: Link Mua Hang (none) -> https://thegioiic.com/products/3296w-203-bien-tro-20k-ohm-t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
Changed lines of the file:
@@
 F 2 "VinhTho_Lib:VR-3362P" H 12125 3325 50  0001 C CNN
 F 3 "https://thegioiic.com/products/3296w-203-bien-tro-20k-ohm-tinh-chinh-top" H 12125 3325 50  0001 C CNN
+F 4 "https://thegioiic.com/products/3296w-203-bien-tro-20k-ohm-tinh-chinh-top" H 12125 3325 50  0001 C CNN "Link Mua Hang"
 	1    12125 3325
 	1    0    0    -1
@@
 F 2 "VinhTho_Lib:MORNSUN-A2412S-2W" H 14600 7256 60  0001 C CIN
 F 3 "https://banlinhkien.shop/module-nguon-cach-ly-a2412s-2w-mornsun" H 14600 6925 60  0001 C CNN
+F 4 "https://banlinhkien.shop/module-nguon-cach-ly-a2412s-2w-mornsun" H 14600 6925 50  0001 C CNN "Link Mua Hang"
 	1    14600 6925
 	-1   0    0    -1
@@
 F 2 "VinhTho_Lib:TO-252-2" H 15825 1300 50  0001 C CNN
 F 3 "https://banlinhkien.com/d409-to252-mosfet-pch-26a-60v-p6650593.html" H 15625 1200 50  0001 C CNN
+F 4 "https://banlinhkien.com/d409-to252-mosfet-pch-26a-60v-p6650593.html" H 15625 1200 50  0001 C CNN "Link Mua Hang"
 	1    15625 1200
 	0    -1   1    0
@@
 F 0 "IC2" H 9975 9744 40  0000 C CNN
 F 1 "6N137" H 9975 9668 40  0000 C CNN
-F 2 "VinhTho_Lib:Diodes_PSOP-8" H 9810 9165 29  0001 C CNN
+F 2 "ph_kicad_lib:SMDIP-8_W9.53mm" H 9810 9165 29  0001 C CNN
 F 3 "https://banlinhkien.com/6n137-sop8-opto-10mbits-p6650639.html" H 9761 9629 60  0001 C CNN
 F 4 "https://banlinhkien.com/6n137-sop8-opto-10mbits-p6650639.html" H 9975 9400 50  0001 C CNN "Link Mua Hang"

Commit message: Update README
Parts:
- BT1: symbol master-node-rescue:Battery_Cell -> ph_door_fume_hood_controller_hw-rescue:Battery_Cell-master-node-rescue
- C1, C10, C11, C12, C13, C14, C15, C16, C17, C18, C19, C2, C20, C21, C22, C23, C24, C25, C26, C28, C29, C3, C30, C31, C33, C35, C36, C37, C38, C4, C40, C42, C43, C45, C46, C47, C48, C49, C50, C51, C52, C6, C7, C8, C9: symbol master-node-rescue:C -> ph_door_fume_hood_controller_hw-rescue:C-master-node-rescue
- C27, C32, C34, C39, C41, C44, C5: symbol master-node-rescue:CP1 -> ph_door_fume_hood_controller_hw-rescue:CP1-master-node-rescue
- D1, D14, D2, D4, D5, D6, D8: symbol master-node-rescue:LED -> ph_door_fume_hood_controller_hw-rescue:LED-master-node-rescue
- D10, D16, D22, D30: symbol ph_door_fume_hood_controller_hw-rescue:D_ALT-Device -> ph_door_fume_hood_controller_hw-rescue:D_ALT-Device-ph_door_fume_hood_controller_hw-rescue
- D11: symbol stm32_st7920_lcd_hw-rescue:TVS-nhantt-kicad-lib -> ph_door_fume_hood_controller_hw-rescue:TVS-nhantt-kicad-lib-stm32_st7920_lcd_hw-rescue
- D12, D17, D18, D19, D20, D24, D27, D28, D29, D31, D32, D33: symbol ph_door_fume_hood_controller_hw-rescue:D_Zener_ALT-Device -> ph_door_fume_hood_controller_hw-rescue:D_Zener_ALT-Device-ph_door_fume_hood_controller_hw-rescue
- D13, D7, D9: symbol master-node-rescue:D_ALT -> ph_door_fume_hood_controller_hw-rescue:D_ALT-master-node-rescue
- D15: symbol ph_door_fume_hood_controller_hw-rescue:D-Device -> ph_door_fume_hood_controller_hw-rescue:D-Device-ph_door_fume_hood_controller_hw-rescue
- D21, D23, D25: symbol ph_door_fume_hood_controller_hw-rescue:D_TVS-Device -> ph_door_fume_hood_controller_hw-rescue:D_TVS-Device-ph_door_fume_hood_controller_hw-rescue
- D26: symbol ph_door_fume_hood_controller_hw-rescue:D_Schottky-Device -> ph_door_fume_hood_controller_hw-rescue:D_Schottky-Device-ph_door_fume_hood_controller_hw-rescue
- D3: symbol ph_door_fume_hood_controller_hw-rescue:1N4148-Diode -> ph_door_fume_hood_controller_hw-rescue:1N4148-Diode-ph_door_fume_hood_controller_hw-rescue
- F1, F2, F3, F4, F5, F6, F7: symbol ph_door_fume_hood_controller_hw-rescue:Fuse-Device -> ph_door_fume_hood_controller_hw-rescue:Fuse-Device-ph_door_fume_hood_controller_hw-rescue
- IC1, IC2: symbol ph_door_fume_hood_controller_hw-rescue:6N137-nhantt-kicad-lib -> ph_door_fume_hood_controller_hw-rescue:6N137-nhantt-kicad-lib-ph_door_fume_hood_controller_hw-rescue
- J1, J10, J14, J15, J4: symbol ph_door_fume_hood_controller_hw-rescue:Conn_01x03-Connector_Generic -> ph_door_fume_hood_controller_hw-rescue:Conn_01x03-Connector_Generic-ph_door_fume_hood_controller_hw-rescue
- J11, J13, J6, J9: symbol ph_door_fume_hood_controller_hw-rescue:Conn_01x02-Connector_Generic -> ph_door_fume_hood_controller_hw-rescue:Conn_01x02-Connector_Generic-ph_door_fume_hood_controller_hw-rescue
- J12, J7: symbol ph_door_fume_hood_controller_hw-rescue:Conn_01x06-Connector_Generic -> ph_door_fume_hood_controller_hw-rescue:Conn_01x06-Connector_Generic-ph_door_fume_hood_controller_hw-rescue
- J2, J5: symbol ph_door_fume_hood_controller_hw-rescue:Conn_01x04-Connector_Generic -> ph_door_fume_hood_controller_hw-rescue:Conn_01x04-Connector_Generic-ph_door_fume_hood_controller_hw-rescue
- J3: symbol master-node-rescue:CONN_01X04 -> ph_door_fume_hood_controller_hw-rescue:CONN_01X04-master-node-rescue
- J8: symbol master-node-rescue:USB_OTG -> ph_door_fume_hood_controller_hw-rescue:USB_OTG-master-node-rescue
- L1: symbol master-node-rescue:L_Small -> ph_door_fume_hood_controller_hw-rescue:L_Small-master-node-rescue
- L2: symbol ph_door_fume_hood_controller_hw-rescue:L_Core_Ferrite-Device -> ph_door_fume_hood_controller_hw-rescue:L_Core_Ferrite-Device-ph_door_fume_hood_controller_hw-rescue
- LS1: symbol ph_door_fume_hood_controller_hw-rescue:Speaker-Device -> ph_door_fume_hood_controller_hw-rescue:Speaker-Device-ph_door_fume_hood_controller_hw-rescue
- M1: symbol ph_door_fume_hood_controller_hw-rescue:DC-DC-24-5V-200mA-nhantt-kicad-lib -> ph_door_fume_hood_controller_hw-rescue:DC-DC-24-5V-200mA-nhantt-kicad-lib-ph_door_fume_hood_controller_hw-rescue
- M2: symbol ph_door_fume_hood_controller_hw-rescue:MORSUN_485-nhantt-kicad-lib -> ph_door_fume_hood_controller_hw-rescue:MORSUN_485-nhantt-kicad-lib-ph_door_fume_hood_controller_hw-rescue
- Q1, Q8: symbol master-node-rescue:C1815 -> ph_door_fume_hood_controller_hw-rescue:C1815-master-node-rescue
- Q10: symbol ph_door_fume_hood_controller_hw-rescue:A1015-nhantt-kicad-lib -> ph_door_fume_hood_controller_hw-rescue:A1015-nhantt-kicad-lib-ph_door_fume_hood_controller_hw-rescue
- Q11, Q4, Q6, Q7, Q9: symbol ph_door_fume_hood_controller_hw-rescue:Q_NMOS_GSD-Device -> ph_door_fume_hood_controller_hw-rescue:Q_NMOS_GSD-Device-ph_door_fume_hood_controller_hw-rescue
- Q2: symbol ph_door_fume_hood_controller_hw-rescue:Q_PMOS_GDS-Device -> ph_door_fume_hood_controller_hw-rescue:Q_PMOS_GDS-Device-ph_door_fume_hood_controller_hw-rescue
- Q3: symbol ph_door_fume_hood_controller_hw-rescue:Q_NMOS_GSD-mcu_water_sample_hw-rescue -> ph_door_fume_hood_controller_hw-rescue:Q_NMOS_GSD-mcu_water_sample_hw-rescue-ph_door_fume_hood_controller_hw-rescue
- Q5: symbol ph_door_fume_hood_controller_hw-rescue:C1815-nhantt-kicad-lib -> ph_door_fume_hood_controller_hw-rescue:C1815-nhantt-kicad-lib-ph_door_fume_hood_controller_hw-rescue
- R1, R10, R11, R14, R15, R16, R17, R2, R21, R22, R23, R24, R27, R28, R29, R3, R30, R31, R32, R34, R35, R36, R37, R38, R39, R40, R41, R42, R43, R44, R45, R47, R49, R52, R53, R54, R55, R56, R57, R58, R64, R66, R68, R69, R7, R71, R73, R74, R79, R8, R82, R84, R85, R86, R87, R88, R9, R94, R95: symbol master-node-rescue:R -> ph_door_fume_hood_controller_hw-rescue:R-master-node-rescue
- R12, R13, R18, R19, R20, R26, R33, R4, R46, R48, R50, R51, R6, R61, R62, R63, R65, R67, R70, R72, R75, R76, R77, R78, R80, R81, R83, R89, R90, R91, R92, R93, R96: symbol ph_door_fume_hood_controller_hw-rescue:R-Device -> ph_door_fume_hood_controller_hw-rescue:R-Device-ph_door_fume_hood_controller_hw-rescue
- R59, R60: symbol ph_door_fume_hood_controller_hw-rescue:R_US-Device -> ph_door_fume_hood_controller_hw-rescue:R_US-Device-ph_door_fume_hood_controller_hw-rescue
- RN1: symbol ph_door_fume_hood_controller_hw-rescue:R_Pack04-Device -> ph_door_fume_hood_controller_hw-rescue:R_Pack04-Device-ph_door_fume_hood_controller_hw-rescue
- RV1: symbol ph_door_fume_hood_controller_hw-rescue:POT-PH_LIB -> ph_door_fume_hood_controller_hw-rescue:POT-PH_LIB-ph_door_fume_hood_controller_hw-rescue
- U1: symbol ph_door_fume_hood_controller_hw-rescue:74HC123-74xx -> ph_door_fume_hood_controller_hw-rescue:74HC123-74xx-ph_door_fume_hood_controller_hw-rescue
- U10, U13, U14, U16, U17, U18, U19, U20, U21, U22, U23, U3, U4, U6: symbol ph_door_fume_hood_controller_hw-rescue:PC817-Isolator -> ph_door_fume_hood_controller_hw-rescue:PC817-Isolator-ph_door_fume_hood_controller_hw-rescue
- U11: symbol ph_door_fume_hood_controller_hw-rescue:MCP4725-nhantt-kicad-lib -> ph_door_fume_hood_controller_hw-rescue:MCP4725-nhantt-kicad-lib-ph_door_fume_hood_controller_hw-rescue
- U12, U8: symbol master-node-rescue:ASM1117 -> ph_door_fume_hood_controller_hw-rescue:ASM1117-master-node-rescue
- U15: symbol ph_door_fume_hood_controller_hw-rescue:LM358-Amplifier_Operational -> ph_door_fume_hood_controller_hw-rescue:LM358-Amplifier_Operational-ph_door_fume_hood_controller_hw-rescue
- U2: symbol ph_door_fume_hood_controller_hw-rescue:AD8601-nhantt-kicad-lib -> ph_door_fume_hood_controller_hw-rescue:AD8601-nhantt-kicad-lib-ph_door_fume_hood_controller_hw-rescue
- U5: symbol ph_door_fume_hood_controller_hw-rescue:TB6600-nhantt-kicad-lib -> ph_door_fume_hood_controller_hw-rescue:TB6600-nhantt-kicad-lib-ph_door_fume_hood_controller_hw-rescue
- U7: symbol master-node-rescue:STM32F103C8 -> ph_door_fume_hood_controller_hw-rescue:STM32F103C8-master-node-rescue
- U9: symbol ph_door_fume_hood_controller_hw-rescue:XL4015-nhantt-kicad-lib -> ph_door_fume_hood_controller_hw-rescue:XL4015-nhantt-kicad-lib-ph_door_fume_hood_controller_hw-rescue
- Y1, Y2: symbol master-node-rescue:Crystal -> ph_door_fume_hood_controller_hw-rescue:Crystal-master-node-rescue
