File: ph_door_fume_hood_controller_hw/ph_door_fume_hood_controller_hw.kicad_pcb (KiCad board)
At the start: 2 copper layers, 3 parts, among them J2 Conn_01x10, U4 STM32F103C8

Commit message: Darwing board fume hood
Parts:
- removed J2: Conn_01x10, nhantt-kicad-lib:Terminal-3.81-10pin
- removed OLED1: Conn_01x07, nhantt-kicad-lib:oled1.3_spi
- removed U4: STM32F103C8, nhantt-kicad-lib:LQFP-48_7x7mm_Pitch0.5mm

Commit message: Layoutting board fume_hood
Parts:
- added BT1: 3V3, VinhTho_Lib:BT3V3, F.Cu at (82.6, -87.9)
- added C1: 100nF, Capacitor_SMD:C_0805_2012Metric_Pad1.15x1.40mm_HandSolder, F.Cu at (259.4, 82.8)
- added C10: 100nF, Capacitor_SMD:C_0805_2012Metric_Pad1.15x1.40mm_HandSolder, F.Cu at (159.6, -53.3)
- added C11: 100nF, Capacitor_SMD:C_0805_2012Metric_Pad1.15x1.40mm_HandSolder, F.Cu at (168.3, -62.4)
- added C12: 100nF, Capacitor_SMD:C_0805_2012Metric_Pad1.15x1.40mm_HandSolder, F.Cu at (125.9, -20.0)
- added C13: 10uF, Capacitor_SMD:C_1206_3216Metric_Pad1.42x1.75mm_HandSolder, F.Cu at (37.0, -13.6)
- added C14: 1uF, Capacitor_SMD:C_0805_2012Metric_Pad1.15x1.40mm_HandSolder, F.Cu at (171.5, -67.8)
- added C15: 100nF, Capacitor_SMD:C_0805_2012Metric_Pad1.15x1.40mm_HandSolder, F.Cu at (221.1, 83.8)
- added C16: C, Capacitor_SMD:C_0805_2012Metric_Pad1.15x1.40mm_HandSolder, F.Cu at (201.0, -99.0)
- added C17: 100nF, Capacitor_SMD:C_0805_2012Metric_Pad1.15x1.40mm_HandSolder, F.Cu at (162.1, -56.3)
- added C18: 1.5uF, Capacitor_SMD:C_0805_2012Metric_Pad1.15x1.40mm_HandSolder, F.Cu at (259.4, 66.5)
- added C19: 100nF, Capacitor_SMD:C_0805_2012Metric_Pad1.15x1.40mm_HandSolder, F.Cu at (116.4, -13.8)
- added C2: 4.7uF, Capacitor_SMD:C_1206_3216Metric_Pad1.42x1.75mm_HandSolder, F.Cu at (259.4, 80.5)
- added C20: 100nF, Capacitor_SMD:C_0805_2012Metric_Pad1.15x1.40mm_HandSolder, F.Cu at (234.0, 46.0)
- added C21: 22pF, Capacitor_SMD:C_0805_2012Metric_Pad1.15x1.40mm_HandSolder, F.Cu at (147.6, -44.0)
- added C22: 100nF, Capacitor_SMD:C_0805_2012Metric_Pad1.15x1.40mm_HandSolder, F.Cu at (179.3, -77.1)
- added C23: 22pF, Capacitor_SMD:C_0805_2012Metric_Pad1.15x1.40mm_HandSolder, F.Cu at (121.1, -16.7)
- added C24: 22pF, Capacitor_SMD:C_0805_2012Metric_Pad1.15x1.40mm_HandSolder, F.Cu at (188.5, -84.3)
- added C25: 22pF, Capacitor_SMD:C_0805_2012Metric_Pad1.15x1.40mm_HandSolder, F.Cu at (141.6, -37.7)
- added C26: 1uF, Capacitor_SMD:C_0805_2012Metric_Pad1.15x1.40mm_HandSolder, F.Cu at (243.9, 36.8)
- added C27: 330uF/25V, Capacitor_SMD:C_1210_3225Metric_Pad1.42x2.65mm_HandSolder, F.Cu at (246.7, 36.8)
- added C28: 1uF, Capacitor_SMD:C_0805_2012Metric_Pad1.15x1.40mm_HandSolder, F.Cu at (261.7, 25.1)
- added C29: 100nF, Capacitor_SMD:C_0805_2012Metric_Pad1.15x1.40mm_HandSolder, F.Cu at (214.7, 27.2)
- added C3: 4.7uF, Capacitor_SMD:C_1206_3216Metric_Pad1.42x1.75mm_HandSolder, F.Cu at (221.1, 86.1)
- added C30: 10uF, Capacitor_SMD:C_0805_2012Metric_Pad1.15x1.40mm_HandSolder, F.Cu at (216.7, 27.2)
- added C31: 1uF, Capacitor_SMD:C_0805_2012Metric_Pad1.15x1.40mm_HandSolder, F.Cu at (261.7, 22.8)
- added C32: 220uF/50V, Capacitor_SMD:C_1210_3225Metric_Pad1.42x2.65mm_HandSolder, F.Cu at (261.7, 19.8)
- added C33: 100nF, Capacitor_SMD:C_0805_2012Metric_Pad1.15x1.40mm_HandSolder, F.Cu at (201.5, 27.2)
- added C34: 100uF/16V, Capacitor_SMD:C_1210_3225Metric_Pad1.42x2.65mm_HandSolder, F.Cu at (204.3, 27.2)
- added C35: 100nF, Capacitor_SMD:C_0805_2012Metric_Pad1.15x1.40mm_HandSolder, F.Cu at (178.1, 109.2)
- added C36: 100nF, Capacitor_SMD:C_0805_2012Metric_Pad1.15x1.40mm_HandSolder, F.Cu at (173.8, -56.0)
- added C37: 100nF, Capacitor_SMD:C_0805_2012Metric_Pad1.15x1.40mm_HandSolder, F.Cu at (178.1, 116.8)
- added C38: 100nF, Capacitor_SMD:C_0805_2012Metric_Pad1.15x1.40mm_HandSolder, F.Cu at (211.2, 115.8)
- added C39: 330uF/25V, Capacitor_SMD:C_1210_3225Metric_Pad1.42x2.65mm_HandSolder, F.Cu at (214.0, 115.8)
- added C4: 100nF, Capacitor_SMD:C_0805_2012Metric_Pad1.15x1.40mm_HandSolder, F.Cu at (221.1, 88.6)
- added C40: 100nF, Capacitor_SMD:C_0805_2012Metric_Pad1.15x1.40mm_HandSolder, F.Cu at (192.9, 118.6)
- added C41: 47uF, Capacitor_SMD:C_1210_3225Metric_Pad1.42x2.65mm_HandSolder, F.Cu at (195.7, 118.6)
- added C42: 100nF, Capacitor_SMD:C_0805_2012Metric_Pad1.15x1.40mm_HandSolder, F.Cu at (53.2, 82.0)
- added C43: 100nF, Capacitor_SMD:C_0805_2012Metric_Pad1.15x1.40mm_HandSolder, F.Cu at (217.8, 115.8)
- added C44: 330uF/25V, Capacitor_SMD:C_1210_3225Metric_Pad1.42x2.65mm_HandSolder, F.Cu at (220.6, 115.8)
- added C45: 100nF, Capacitor_SMD:C_0805_2012Metric_Pad1.15x1.40mm_HandSolder, F.Cu at (178.1, 119.4)
- added C46: 100nF, Capacitor_SMD:C_0805_2012Metric_Pad1.15x1.40mm_HandSolder, F.Cu at (180.2, 127.2)
- added C47: 100nF, Capacitor_SMD:C_0805_2012Metric_Pad1.15x1.40mm_HandSolder, F.Cu at (53.2, 75.4)
- added C48: 100nF, Capacitor_SMD:C_0805_2012Metric_Pad1.15x1.40mm_HandSolder, F.Cu at (173.3, -70.8)
- added C49: 100nF, Capacitor_SMD:C_0805_2012Metric_Pad1.15x1.40mm_HandSolder, F.Cu at (53.2, 68.8)
- added C5: 470uF/50V, Capacitor_SMD:C_1210_3225Metric_Pad1.42x2.65mm_HandSolder, F.Cu at (220.0, 71.9)
- added C50: 100nF, Capacitor_SMD:C_0805_2012Metric_Pad1.15x1.40mm_HandSolder, F.Cu at (201.0, -101.9)
- added C51: 100nF, Capacitor_SMD:C_0805_2012Metric_Pad1.15x1.40mm_HandSolder, F.Cu at (53.2, 62.2)
- added C52: 100nF, Capacitor_SMD:C_0805_2012Metric_Pad1.15x1.40mm_HandSolder, F.Cu at (116.4, -16.7)
- added C6: 4.7nF, Capacitor_SMD:C_0805_2012Metric_Pad1.15x1.40mm_HandSolder, F.Cu at (153.7, -47.0)
- added C7: 100nF, Capacitor_SMD:C_0805_2012Metric_Pad1.15x1.40mm_HandSolder, F.Cu at (220.0, 65.9)
- added C8: 100nF, Capacitor_SMD:C_0805_2012Metric_Pad1.15x1.40mm_HandSolder, F.Cu at (220.0, 68.6)
- added C9: 4.7nF, Capacitor_SMD:C_0805_2012Metric_Pad1.15x1.40mm_HandSolder, F.Cu at (196.5, -90.0)
- added D1: LED, LED_SMD:LED_0805_2012Metric_Pad1.15x1.40mm_HandSolder, F.Cu at (251.3, 85.6)
- added D10: D_ALT, VinhTho_Lib:D_SMA_Standard, F.Cu at (187.5, 51.5)
- added D11: TVS, VinhTho_Lib:D_SMA_Standard, F.Cu at (263.0, 38.6)
- added D12: 10V, VinhTho_Lib:SOD-80, F.Cu at (168.0, 55.6)
- added D13: D_ALT, VinhTho_Lib:D_SOD-323F, F.Cu at (82.4, -49.1)
- added D14: LED, LED_SMD:LED_0805_2012Metric_Pad1.15x1.40mm_HandSolder, F.Cu at (209.4, 104.1)
- added D15: D, VinhTho_Lib:D_SOD-323F, F.Cu at (82.1, -65.5)
- added D16: D_ALT, VinhTho_Lib:D_SMA_Standard, F.Cu at (187.5, 63.0)
- added D17: D_Zener_ALT, VinhTho_Lib:SOD-80, F.Cu at (37.3, 82.2)
- added D18: 10V, VinhTho_Lib:SOD-80, F.Cu at (168.0, 67.0)
- added D19: D_Zener_ALT, VinhTho_Lib:SOD-80, F.Cu at (37.3, 75.7)
- added D2: LED, LED_SMD:LED_0805_2012Metric_Pad1.15x1.40mm_HandSolder, F.Cu at (251.3, 63.7)
- added D20: D_Zener_ALT, VinhTho_Lib:SOD-80, F.Cu at (37.3, 96.6)
- added D21: D_TVS, VinhTho_Lib:D_SMA_Standard, F.Cu at (149.7, 132.3)
- added D22: D_ALT, VinhTho_Lib:D_SMA_Standard, F.Cu at (187.5, 74.7)
- added D23: D_TVS, VinhTho_Lib:D_SMA_Standard, F.Cu at (157.3, 132.3)
- added D24: 10V, VinhTho_Lib:SOD-80, F.Cu at (168.0, 78.7)
- added D25: D_TVS, VinhTho_Lib:D_SMA_Standard, F.Cu at (164.9, 132.3)
- added D26: SS54, VinhTho_Lib:D_SMA_Standard, F.Cu at (234.0, 130.5)
- added D27: D_Zener_ALT, VinhTho_Lib:SOD-80, F.Cu at (37.3, 69.1)
- added D28: D_Zener_ALT, VinhTho_Lib:SOD-80, F.Cu at (169.8, -78.7)
- added D29: 12V, VinhTho_Lib:SOD-80, F.Cu at (215.7, 133.3)
- added D3: 1N4148, Diode_SMD:D_SOD-323_HandSoldering, F.Cu at (53.9, -13.4)
- added D30: D_ALT, VinhTho_Lib:D_SMA_Standard, F.Cu at (187.5, 86.6)
- added D31: D_Zener_ALT, VinhTho_Lib:SOD-80, F.Cu at (37.3, 62.5)
- added D32: D_Zener_ALT, VinhTho_Lib:SOD-80, F.Cu at (134.5, -49.0)
- added D33: 10V, VinhTho_Lib:SOD-80, F.Cu at (168.0, 90.7)
- added D4: LED, LED_SMD:LED_0805_2012Metric_Pad1.15x1.40mm_HandSolder, F.Cu at (82.3, -46.1)
- added D5: LED, LED_SMD:LED_0805_2012Metric_Pad1.15x1.40mm_HandSolder, F.Cu at (68.4, -13.3)
- added D6: LED, LED_SMD:LED_0805_2012Metric_Pad1.15x1.40mm_HandSolder, F.Cu at (63.6, -13.3)
- added D7: D_ALT, VinhTho_Lib:D_SMA_Standard, F.Cu at (218.8, 76.4)
- added D8: LED, LED_SMD:LED_0805_2012Metric_Pad1.15x1.40mm_HandSolder, F.Cu at (215.5, 21.1)
- added D9: D_ALT, VinhTho_Lib:D_SMA_Standard, F.Cu at (263.2, 29.4)
- added F1: Fuse, VinhTho_Lib:Fuse_SMD1812, F.Cu at (263.2, 34.0)
- added F2: Fuse, VinhTho_Lib:Fuse_SMD1812, F.Cu at (187.5, 56.1)
- added F3: Fuse, VinhTho_Lib:Fuse_SMD1812, F.Cu at (187.5, 67.5)
- added F4: Fuse, VinhTho_Lib:Fuse_SMD1812, F.Cu at (187.5, 79.2)
- added F5: Fuse, VinhTho_Lib:Fuse_SMD1812, F.Cu at (153.5, 138.4)
- added F6: Fuse, VinhTho_Lib:Fuse_SMD1812, F.Cu at (160.9, 138.4)
- added F7: Fuse, VinhTho_Lib:Fuse_SMD1812, F.Cu at (187.5, 91.2)
- added IC1: 6N137, VinhTho_Lib:Diodes_PSOP-8, F.Cu at (207.3, 78.2)
- added IC2: 6N137, VinhTho_Lib:Diodes_PSOP-8, F.Cu at (199.2, 130.8)
- added J1: Conn_01x03, VinhTho_Lib:TerminalBlock-WAGO-3P, F.Cu at (95.3, -61.4)
- added J10: Conn_01x03, VinhTho_Lib:TerminalBlock-WAGO-3P, F.Cu at (17.4, 98.5)
- added J11: Conn_01x02, VinhTho_Lib:TerminalBlock_WAGO-236_2Stift_R5mm_2pol, F.Cu at (157.1, 152.6)
- added J12: Conn_01x06, VinhTho_Lib:TerminalBlock-WAGO-6P, F.Cu at (16.3, 60.9)
- added J13: Conn_01x02, VinhTho_Lib:TerminalBlock_WAGO-236_2Stift_R5mm_2pol, F.Cu at (246.0, 128.8)
- added J14: Conn_01x03, VinhTho_Lib:TerminalBlock-WAGO-3P, F.Cu at (17.4, 117.1)
- added J15: Conn_01x03, VinhTho_Lib:TerminalBlock-WAGO-3P, F.Cu at (17.4, 135.6)
- added J2: Conn_01x04, VinhTho_Lib:Domino-5.08mm_4pol, F.Cu at (276.7, 75.7)
- added J3: CONN_01X04, Connector_PinHeader_2.54mm:PinHeader_1x04_P2.54mm_Vertical, F.Cu at (147.9, -16.3)
- added J4: Conn_01x03, VinhTho_Lib:TerminalBlock-WAGO-3P, F.Cu at (145.4, -96.3)
- added J5: Conn_01x03, VinhTho_Lib:TerminalBlock-WAGO-3P, F.Cu at (114.7, -89.5)
- added J6: Conn_01x02, VinhTho_Lib:TerminalBlock_WAGO-236_2Stift_R5mm_2pol, F.Cu at (278.5, 31.5)
- added J7: Conn_01x06, VinhTho_Lib:TerminalBlock-WAGO-6P, F.Cu at (191.3, 24.4)
- added J8: USB_OTG, VinhTho_Lib:USB_Micro-B, F.Cu at (124.8, -61.2)
- added J9: Conn_01x02, VinhTho_Lib:TerminalBlock_WAGO-236_2Stift_R5mm_2pol, F.Cu at (177.4, 139.9)
- added L1: L_Small, Inductor_SMD:L_0805_2012Metric_Pad1.15x1.40mm_HandSolder, F.Cu at (162.1, -59.2)
- added L2: 180uH/5A, VinhTho_Lib:L181-5A, F.Cu at (232.2, 27.9)
- added LS1: Speaker, Buzzer_Beeper:Buzzer_15x7.5RM7.6, F.Cu at (109.2, -64.5)
- added M1: DC-DC-24-12V-200mA, VinhTho_Lib:MORNSUN-A2412S-2W, F.Cu at (214.5, 108.7)
- added M2: MORSUN_485, VinhTho_Lib:MORSUN_485, F.Cu at (157.1, 117.3)
- added Q1: C1815, VinhTho_Lib:SOT-23, F.Cu at (236.6, 52.8)
- added Q10: A1015, VinhTho_Lib:SOT-23, F.Cu at (210.9, 132.3)
- added Q11: Q_NMOS_GDS, VinhTho_Lib:TO-252-2, F.Cu at (176.6, 89.6)
- added Q2: Q_PMOS_GDS, VinhTho_Lib:TO-252-2, F.Cu at (226.4, 54.8)
- added Q3: Q_NMOS_GDS, VinhTho_Lib:TO-252-2, F.Cu at (251.5, 54.8)
- added Q4: Q_NMOS_GDS, VinhTho_Lib:TO-252-2, F.Cu at (176.6, 54.6)
- added Q5: C1815, VinhTho_Lib:SOT-23, F.Cu at (172.5, -46.5)
- added Q6: Q_NMOS_GDS, VinhTho_Lib:TO-252-2, F.Cu at (176.6, 66.0)
- added Q7: Q_NMOS_GDS, VinhTho_Lib:TO-252-2, F.Cu at (176.6, 77.7)
- added Q8: C1815, VinhTho_Lib:SOT-23, F.Cu at (210.9, 128.8)
- added Q9: Q_NMOS_GDS, VinhTho_Lib:TO-252-2, F.Cu at (225.4, 130.8)
- added R1: 2.2k, Resistor_SMD:R_0805_2012Metric_Pad1.15x1.40mm_HandSolder, F.Cu at (237.6, 56.6)
- added R10: 10k, Resistor_SMD:R_0805_2012Metric_Pad1.15x1.40mm_HandSolder, F.Cu at (212.4, 78.2)
- added R11: 1k, Resistor_SMD:R_0805_2012Metric_Pad1.15x1.40mm_HandSolder, F.Cu at (251.3, 61.5)
- added R12: 1k, Resistor_SMD:R_0805_2012Metric_Pad1.15x1.40mm_HandSolder, F.Cu at (201.3, 64.5)
- added R13: 10k, Resistor_SMD:R_0805_2012Metric_Pad1.15x1.40mm_HandSolder, F.Cu at (213.7, 64.5)
- added R14: 100R, Resistor_SMD:R_0805_2012Metric_Pad1.15x1.40mm_HandSolder, F.Cu at (202.0, 78.0)
- added R15: 10k, Resistor_SMD:R_0805_2012Metric_Pad1.15x1.40mm_HandSolder, F.Cu at (244.2, 93.2)
- added R16: 10k, Resistor_SMD:R_0805_2012Metric_Pad1.15x1.40mm_HandSolder, F.Cu at (235.0, 93.2)
- added R17: 10k, Resistor_SMD:R_0805_2012Metric_Pad1.15x1.40mm_HandSolder, F.Cu at (239.6, 93.2)
- added R18: 51R, Resistor_SMD:R_0805_2012Metric_Pad1.15x1.40mm_HandSolder, F.Cu at (173.0, -64.9)
- added R19: 51R, Resistor_SMD:R_0805_2012Metric_Pad1.15x1.40mm_HandSolder, F.Cu at (164.3, -53.3)
- added R2: 10k, Resistor_SMD:R_0805_2012Metric_Pad1.15x1.40mm_HandSolder, F.Cu at (235.3, 56.6)
- added R20: 100R, Resistor_SMD:R_0805_2012Metric_Pad1.15x1.40mm_HandSolder, F.Cu at (193.2, -82.4)
- added R21: 10k, Resistor_SMD:R_0805_2012Metric_Pad1.15x1.40mm_HandSolder, F.Cu at (241.9, 93.2)
- added R22: 10k, Resistor_SMD:R_0805_2012Metric_Pad1.15x1.40mm_HandSolder, F.Cu at (232.7, 93.2)
- added R23: 10k, Resistor_SMD:R_0805_2012Metric_Pad1.15x1.40mm_HandSolder, F.Cu at (237.3, 93.2)
- added R24: 10k, Resistor_SMD:R_0805_2012Metric_Pad1.15x1.40mm_HandSolder, F.Cu at (213.4, 71.6)
- added R25: 0R, Resistor_SMD:R_0805_2012Metric_Pad1.15x1.40mm_HandSolder, F.Cu at (140.1, -18.8)
- added R26: 124k, Resistor_SMD:R_0805_2012Metric_Pad1.15x1.40mm_HandSolder, F.Cu at (190.5, -68.3)
- added R27: 100R, Resistor_SMD:R_0805_2012Metric_Pad1.15x1.40mm_HandSolder, F.Cu at (201.3, 71.6)
- added R28: 0.62R, Resistor_SMD:R_0805_2012Metric_Pad1.15x1.40mm_HandSolder, F.Cu at (251.3, 76.9)
- added R29: 0.62R, Resistor_SMD:R_0805_2012Metric_Pad1.15x1.40mm_HandSolder, F.Cu at (251.3, 79.2)
- added R3: 1k, Resistor_SMD:R_0805_2012Metric_Pad1.15x1.40mm_HandSolder, F.Cu at (251.3, 87.9)
- added R30: 0.62R, Resistor_SMD:R_0805_2012Metric_Pad1.15x1.40mm_HandSolder, F.Cu at (251.3, 74.7)
- added R31: 10k, Resistor_SMD:R_0805_2012Metric_Pad1.15x1.40mm_HandSolder, F.Cu at (221.1, 81.5)
- added R32: 10k, Resistor_SMD:R_0805_2012Metric_Pad1.15x1.40mm_HandSolder, F.Cu at (213.4, 84.8)
- added R33: R, Resistor_SMD:R_0805_2012Metric_Pad1.15x1.40mm_HandSolder, F.Cu at (182.8, -71.2)
- added R34: 10k, Resistor_SMD:R_0805_2012Metric_Pad1.15x1.40mm_HandSolder, F.Cu at (242.7, 53.6)
- added R35: 10k, Resistor_SMD:R_0805_2012Metric_Pad1.15x1.40mm_HandSolder, F.Cu at (125.9, -14.1)
- added R36: 1M, Resistor_SMD:R_0805_2012Metric_Pad1.15x1.40mm_HandSolder, F.Cu at (259.4, 64.2)
- added R37: 100R, Resistor_SMD:R_0805_2012Metric_Pad1.15x1.40mm_HandSolder, F.Cu at (201.3, 84.8)
- added R38: 15k, Resistor_SMD:R_0805_2012Metric_Pad1.15x1.40mm_HandSolder, F.Cu at (247.2, 46.0)
- added R39: 0.62R, Resistor_SMD:R_0805_2012Metric_Pad1.15x1.40mm_HandSolder, F.Cu at (251.3, 72.4)
- added R4: 0R, Resistor_SMD:R_0805_2012Metric_Pad1.15x1.40mm_HandSolder, F.Cu at (166.8, -59.3)
- added R40: 0.62R, Resistor_SMD:R_0805_2012Metric_Pad1.15x1.40mm_HandSolder, F.Cu at (251.3, 70.1)
- added R41: 0.62R, Resistor_SMD:R_0805_2012Metric_Pad1.15x1.40mm_HandSolder, F.Cu at (251.3, 67.8)
- added R42: 0R, Resistor_SMD:R_0805_2012Metric_Pad1.15x1.40mm_HandSolder, F.Cu at (242.7, 56.6)
- added R43: 51k, Resistor_SMD:R_0805_2012Metric_Pad1.15x1.40mm_HandSolder, F.Cu at (251.3, 81.5)
- added R44: 10k, Resistor_SMD:R_0805_2012Metric_Pad1.15x1.40mm_HandSolder, F.Cu at (152.3, -41.1)
- added R45: 1k, Resistor_SMD:R_0805_2012Metric_Pad1.15x1.40mm_HandSolder, F.Cu at (215.5, 23.4)
- added R46: 10k, Resistor_SMD:R_0805_2012Metric_Pad1.15x1.40mm_HandSolder, F.Cu at (164.9, 51.5)
- added R47: 13k, Resistor_SMD:R_0805_2012Metric_Pad1.15x1.40mm_HandSolder, F.Cu at (249.5, 36.8)
- added R48: 1k, Resistor_SMD:R_0805_2012Metric_Pad1.15x1.40mm_HandSolder, F.Cu at (158.6, 50.8)
- added R49: 1.5k, Resistor_SMD:R_0805_2012Metric_Pad1.15x1.40mm_HandSolder, F.Cu at (251.8, 36.8)
- added R5: 0R, Resistor_SMD:R_0805_2012Metric_Pad1.15x1.40mm_HandSolder, F.Cu at (176.3, -67.8)
- added R50: 10R, Resistor_SMD:R_0805_2012Metric_Pad1.15x1.40mm_HandSolder, F.Cu at (168.0, 51.8)
- added R51: 10k, Resistor_SMD:R_0805_2012Metric_Pad1.15x1.40mm_HandSolder, F.Cu at (164.9, 56.4)
- added R52: 4.7k, Resistor_SMD:R_0805_2012Metric_Pad1.15x1.40mm_HandSolder, F.Cu at (174.6, 113.5)
- added R53: 4.7k, Resistor_SMD:R_0805_2012Metric_Pad1.15x1.40mm_HandSolder, F.Cu at (174.6, 109.7)
- added R54: 1.5k, Resistor_SMD:R_0805_2012Metric_Pad1.15x1.40mm_HandSolder, F.Cu at (193.5, -79.5)
- added R55: 22R, Resistor_SMD:R_0805_2012Metric_Pad1.15x1.40mm_HandSolder, F.Cu at (169.1, -53.4)
- added R56: 2.2k, Resistor_SMD:R_0805_2012Metric_Pad1.15x1.40mm_HandSolder, F.Cu at (205.3, 104.1)
- added R57: 22R, Resistor_SMD:R_0805_2012Metric_Pad1.15x1.40mm_HandSolder, F.Cu at (193.2, -85.4)
- added R58: R, Resistor_SMD:R_0805_2012Metric_Pad1.15x1.40mm_HandSolder, F.Cu at (178.1, 114.8)
- added R59: 100R/2512, Resistor_SMD:R_2512_6332Metric_Pad1.52x3.35mm_HandSolder, F.Cu at (203.5, 115.8)
- added R6: 1k, Resistor_SMD:R_0805_2012Metric_Pad1.15x1.40mm_HandSolder, F.Cu at (152.3, -44.0)
- added R60: 100R/2512, Resistor_SMD:R_2512_6332Metric_Pad1.52x3.35mm_HandSolder, F.Cu at (207.9, 115.8)
- added R61: 10k, Resistor_SMD:R_0805_2012Metric_Pad1.15x1.40mm_HandSolder, F.Cu at (164.9, 63.0)
- added R62: 10k, Resistor_SMD:R_0805_2012Metric_Pad1.15x1.40mm_HandSolder, F.Cu at (53.2, 79.5)
- added R63: 1k, Resistor_SMD:R_0805_2012Metric_Pad1.15x1.40mm_HandSolder, F.Cu at (158.6, 62.2)
- added R64: 2.2k, Resistor_SMD:R_0805_2012Metric_Pad1.15x1.40mm_HandSolder, F.Cu at (152.6, -31.8)
- added R65: 10R, Resistor_SMD:R_0805_2012Metric_Pad1.15x1.40mm_HandSolder, F.Cu at (168.0, 63.2)
- added R66: 2.2k, Resistor_SMD:R_0805_2012Metric_Pad1.15x1.40mm_HandSolder, F.Cu at (37.3, 78.9)
- added R67: 10k, Resistor_SMD:R_0805_2012Metric_Pad1.15x1.40mm_HandSolder, F.Cu at (164.9, 67.8)
- added R68: R, Resistor_SMD:R_0805_2012Metric_Pad1.15x1.40mm_HandSolder, F.Cu at (176.1, 127.2)
- added R69: 10k, Resistor_SMD:R_0805_2012Metric_Pad1.15x1.40mm_HandSolder, F.Cu at (173.1, 121.4)
- added R7: 1k, Resistor_SMD:R_0805_2012Metric_Pad1.15x1.40mm_HandSolder, F.Cu at (133.2, -24.7)
- added R70: 10k, Resistor_SMD:R_0805_2012Metric_Pad1.15x1.40mm_HandSolder, F.Cu at (53.2, 72.9)
- added R71: 33k, Resistor_SMD:R_0805_2012Metric_Pad1.15x1.40mm_HandSolder, F.Cu at (173.1, 125.5)
- added R72: 10k, Resistor_SMD:R_0805_2012Metric_Pad1.15x1.40mm_HandSolder, F.Cu at (157.3, -32.2)
- added R73: 2.2k, Resistor_SMD:R_0805_2012Metric_Pad1.15x1.40mm_HandSolder, F.Cu at (37.3, 72.4)
- added R74: 2.2k, Resistor_SMD:R_0805_2012Metric_Pad1.15x1.40mm_HandSolder, F.Cu at (37.3, 93.3)
- added R75: 10k, Resistor_SMD:R_0805_2012Metric_Pad1.15x1.40mm_HandSolder, F.Cu at (164.9, 74.7)
- added R76: 1k, Resistor_SMD:R_0805_2012Metric_Pad1.15x1.40mm_HandSolder, F.Cu at (158.6, 73.6)
- added R77: 10R, Resistor_SMD:R_0805_2012Metric_Pad1.15x1.40mm_HandSolder, F.Cu at (168.0, 74.9)
- added R78: 120R, Resistor_SMD:R_0805_2012Metric_Pad1.15x1.40mm_HandSolder, F.Cu at (157.3, 129.3)
- added R79: 10k, Resistor_SMD:R_0805_2012Metric_Pad1.15x1.40mm_HandSolder, F.Cu at (215.7, 128.5)
- added R8: 1k, Resistor_SMD:R_0805_2012Metric_Pad1.15x1.40mm_HandSolder, F.Cu at (158.5, -49.9)
- added R80: 10k, Resistor_SMD:R_0805_2012Metric_Pad1.15x1.40mm_HandSolder, F.Cu at (164.9, 79.5)
- added R81: 10k, Resistor_SMD:R_0805_2012Metric_Pad1.15x1.40mm_HandSolder, F.Cu at (53.2, 66.3)
- added R82: 10k, Resistor_SMD:R_0805_2012Metric_Pad1.15x1.40mm_HandSolder, F.Cu at (204.6, 130.3)
- added R83: 10k, Resistor_SMD:R_0805_2012Metric_Pad1.15x1.40mm_HandSolder, F.Cu at (193.5, -76.5)
- added R84: 2.2k, Resistor_SMD:R_0805_2012Metric_Pad1.15x1.40mm_HandSolder, F.Cu at (37.3, 65.8)
- added R85: 2.2k, Resistor_SMD:R_0805_2012Metric_Pad1.15x1.40mm_HandSolder, F.Cu at (142.7, -25.9)
- added R86: 2.2k, Resistor_SMD:R_0805_2012Metric_Pad1.15x1.40mm_HandSolder, F.Cu at (206.8, 130.3)
- added R87: 10k, Resistor_SMD:R_0805_2012Metric_Pad1.15x1.40mm_HandSolder, F.Cu at (215.7, 130.8)
- added R88: 100R, Resistor_SMD:R_0805_2012Metric_Pad1.15x1.40mm_HandSolder, F.Cu at (194.1, 130.3)
- added R89: 10k, Resistor_SMD:R_0805_2012Metric_Pad1.15x1.40mm_HandSolder, F.Cu at (164.9, 86.6)
- added R9: 1k, Resistor_SMD:R_0805_2012Metric_Pad1.15x1.40mm_HandSolder, F.Cu at (146.4, -37.7)
- added R90: 1k, Resistor_SMD:R_0805_2012Metric_Pad1.15x1.40mm_HandSolder, F.Cu at (158.6, 85.6)
- added R91: 10k, Resistor_SMD:R_0805_2012Metric_Pad1.15x1.40mm_HandSolder, F.Cu at (53.2, 59.7)
- added R92: 10k, Resistor_SMD:R_0805_2012Metric_Pad1.15x1.40mm_HandSolder, F.Cu at (147.8, -28.9)
- added R93: 10R, Resistor_SMD:R_0805_2012Metric_Pad1.15x1.40mm_HandSolder, F.Cu at (168.0, 86.9)
- added R94: 2.2k, Resistor_SMD:R_0805_2012Metric_Pad1.15x1.40mm_HandSolder, F.Cu at (37.3, 59.2)
- added R95: 2.2k, Resistor_SMD:R_0805_2012Metric_Pad1.15x1.40mm_HandSolder, F.Cu at (166.6, -44.4)
- added R96: 10k, Resistor_SMD:R_0805_2012Metric_Pad1.15x1.40mm_HandSolder, F.Cu at (164.9, 91.4)
- added RN1: R_Network04, Resistor_THT:R_Array_SIP5, F.Cu at (150.7, 76.9)
- added RV1: 20k, VinhTho_Lib:VR1, F.Cu at (243.2, 46.0)
- added U1: 74HC123, VinhTho_Lib:SOIC-16W_5.3x10.2mm_Pitch1.27mm, F.Cu at (259.4, 73.4)
- added U10: PC817, Package_DIP:DIP-4_W7.62mm, F.Cu at (154.8, 53.6)
- added U11: MCP4725, VinhTho_Lib:SOT-23-6_Handsoldering, F.Cu at (178.1, 112.0)
- added U12: ASM1117-3V3, VinhTho_Lib:SOT-223, F.Cu at (195.7, 111.5)
- added U13: PC817, Package_DIP:DIP-4_W7.62mm, F.Cu at (154.8, 65.0)
- added U14: PC817, Package_DIP:DIP-4_W7.62mm, F.Cu at (42.1, 79.5)
- added U15: LM358, Package_SO:SOP-8_3.76x4.96mm_P1.27mm, F.Cu at (178.1, 123.2)
- added U16: PC817, Package_DIP:DIP-4_W7.62mm, F.Cu at (42.1, 72.9)
- added U17: PC817, Package_DIP:DIP-4_W7.62mm, F.Cu at (42.1, 94.1)
- added U18: PC817, Package_DIP:DIP-4_W7.62mm, F.Cu at (154.8, 76.7)
- added U19: PC817, Package_DIP:DIP-4_W7.62mm, F.Cu at (42.1, 66.3)
- added U2: AD8601, VinhTho_Lib:SOT-23-5, F.Cu at (132.6, -81.6)
- added U20: PC817, Package_DIP:DIP-4_W7.62mm, F.Cu at (42.1, 112.1)
- added U21: PC817, Package_DIP:DIP-4_W7.62mm, F.Cu at (154.8, 88.6)
- added U22: PC817, Package_DIP:DIP-4_W7.62mm, F.Cu at (42.1, 59.7)
- added U23: PC817, Package_DIP:DIP-4_W7.62mm, F.Cu at (42.1, 130.8)
- added U3: PC817, Package_DIP:DIP-4_W7.62mm, F.Cu at (203.5, 63.2)
- added U4: PC817, Package_DIP:DIP-4_W7.62mm, F.Cu at (203.5, 70.3)
- added U5: TB6600, VinhTho_Lib:TB6600, F.Cu at (236.6, 76.0)
- added U6: PC817, Package_DIP:DIP-4_W7.62mm, F.Cu at (203.5, 83.5)
- added U7: STM32F103C8, VinhTho_Lib:LQFP-48_7x7mm_Pitch0.5mm, F.Cu at (124.7, -50.4)
- added U8: ASM1117, VinhTho_Lib:SOT-223, F.Cu at (209.9, 27.2)
- added U9: XL4015, Package_TO_SOT_SMD:TO-263-5_TabPin3, F.Cu at (252.8, 25.6)
- added Y1: Crystal, VinhTho_Lib:Crystal_SMD_HC49-SD, F.Cu at (131.5, -76.4)
- added Y2: 32768Mhz, VinhTho_Lib:Crystal_Round_Horizontal_3mm_smd, F.Cu at (81.8, -69.3)

Commit message: Layoutting Board Door-Fume-Hood
Parts:
- J1, J4, J5: footprint VinhTho_Lib:TerminalBlock-WAGO-3P -> Connector_PinSocket_2.54mm:PinSocket_1x03_P2.54mm_Vertical
- J10, J14, J15: footprint VinhTho_Lib:TerminalBlock-WAGO-3P -> VinhTho_Lib:TerminalBlock_WAGO_2.54mm_3P
- moved C50 220.4 mm to (91.5, 89.4), turned to 180 degrees
- moved R83 192.8 mm to (91.5, 87.1), turned to 180 degrees
- moved D28 192.6 mm to (75.6, 89.3)
- moved C9 174.2 mm to (74.5, 34.2), turned to 90 degrees
- moved C16 173.1 mm to (80.6, 25.4), turned to 270 degrees
- moved C48 171.1 mm to (91.5, 79.5), turned to 180 degrees
- moved J5 169.0 mm to (106.5, 79.2)
- moved R95 167.4 mm to (75.8, 96.2)
- moved C24 165.1 mm to (121.7, 66.8), turned to 90 degrees
- moved D32 159.8 mm to (75.8, 99.6)
- moved R20 159.3 mm to (80.6, 30.2), turned to 270 degrees
- moved R26 156.7 mm to (68.7, 30.2), turned to 270 degrees
- moved C14 151.8 mm to (122.8, 75.9), turned to 180 degrees
- moved R57 151.0 mm to (95.1, 29.4), turned to 90 degrees
- moved C11 149.8 mm to (106.5, 74.1), turned to 180 degrees
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Connections:
- D20 pad 1: Net-(D20-Pad1) -> +24V
- D28 pad 1: Net-(D28-Pad1) -> +24V
- D32 pad 1: Net-(D32-Pad1) -> +24V
- R5 pad 2: Net-(R5-Pad2) -> +24V
Routing:
- net +12V: track 0.00 -> 96.3 mm
- net +5V: track 0.00 -> 62.2 mm, vias 0 -> 2
- net /CLK: track 0.00 -> 42.8 mm, vias 0 -> 1
- net Net-(L2-Pad2): track 0.00 -> 35.1 mm
- net /VREF: track 0.00 -> 33.6 mm, vias 0 -> 1
- net Net-(Q3-Pad1): track 0.00 -> 28.4 mm
- net Net-(C5-Pad1): track 0.00 -> 27.1 mm
- net +24V: track 0.00 -> 25.3 mm
- net Net-(R39-Pad2): track 0.00 -> 25.2 mm
- net Net-(R28-Pad2): track 0.00 -> 24.9 mm
- net +12VA: track 0.00 -> 23.8 mm
- net Net-(R43-Pad1): track 0.00 -> 21.8 mm
- net Net-(D1-Pad1): track 0.00 -> 20.9 mm
- net Net-(C28-Pad2): track 0.00 -> 20.9 mm, vias 0 -> 2
- net Net-(D2-Pad1): track 0.00 -> 20.7 mm
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Other:
- board outline added: 166.2 x 133.3 mm

Commit message: Update
Parts:
- F5, F6: moved to B.Cu
- moved LS1 106.8 mm to (124.5, 133.9)
- moved BT1 98.6 mm to (120.1, 147.8), turned to 270 degrees
- moved J9 86.5 mm to (214.9, 145.8), turned to 270 degrees
- moved C40 76.4 mm to (110.6, 42.1)
- moved C41 76.4 mm to (113.4, 42.1)
- moved U12 76.4 mm to (113.4, 35.0)
- moved D14 73.6 mm to (125.6, 30.6)
- moved R56 73.6 mm to (121.5, 30.6)
- moved C38 72.5 mm to (125.1, 43.8)
- moved C39 72.5 mm to (127.8, 43.8)
- moved C43 72.5 mm to (131.7, 43.8)
- moved C44 72.5 mm to (134.4, 43.8)
- moved M1 72.5 mm to (128.4, 36.7)
- moved R59 72.5 mm to (117.4, 43.8)
- moved R60 72.5 mm to (121.8, 43.8)
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Routing:
- net +24V: track 25.3 -> 583.2 mm, vias 0 -> 5
- net +5V: track 62.2 -> 272.2 mm, vias 2 -> 8
- net +3V3: track 11.8 -> 194.9 mm, vias 0 -> 3
- net /CLK: track 42.8 -> 126.0 mm, vias 1 -> 0
- net Net-(J2-Pad2): track 0.00 -> 71.0 mm, vias 0 -> 1
- net Net-(J2-Pad1): track 0.00 -> 68.1 mm, vias 0 -> 1
- net Net-(J2-Pad4): track 0.00 -> 67.7 mm, vias 0 -> 6
- net Net-(J2-Pad3): track 0.00 -> 67.0 mm, vias 0 -> 3
- net /M1: track 0.00 -> 39.1 mm, vias 0 -> 1
- net GND: track 0.00 -> 36.7 mm
- net /PWR_STEP: track 0.00 -> 36.2 mm, vias 0 -> 2
- net /M2: track 0.00 -> 35.9 mm, vias 0 -> 2
- net Net-(D26-Pad2): track 0.00 -> 30.9 mm
- net /M3: track 0.00 -> 30.0 mm, vias 0 -> 1
- net /EN: track 0.00 -> 22.1 mm
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- added copper zone on F.Cu, net +24V
- added copper zone on B.Cu, net +3V3
- added copper zone on F.Cu, net +3V3
- added copper zone on B.Cu, net Net-(D11-Pad1)
- added copper zone on F.Cu, net Net-(D11-Pad1)
- added copper zone on B.Cu, net Net-(F1-Pad1)
- added copper zone on F.Cu, net Net-(F1-Pad1)
- added copper zone on B.Cu, net Net-(J2-Pad3)
- added copper zone on F.Cu, net Net-(J2-Pad3)
- added copper zone on B.Cu, net Net-(J2-Pad4)
- added copper zone on F.Cu, net Net-(J2-Pad4)
Other:
- board size 166.2 x 133.3 mm -> 145.7 x 133.3 mm
- net class Default: clearance 0.2 -> 0.25
- rule trace_clearance: 0.2 -> 0.25
